Commit message: feat: update a1_descpriton add gazebo launch
Signed-off-by: Maciej Krupka <maciej.p.krupka@student.put.poznan.pl>

File: a1_description/xacro/gazebo.xacro (robot description, xacro)
@@ -2,12 +2,12 @@
 <robot>
     <!-- ros_control plugin -->
-    <gazebo>
+    <!-- <gazebo>
         <plugin name="gazebo_ros_control" filename="libgazebo_ros_control.so">
             <robotNamespace>/a1_gazebo</robotNamespace>
             <robotSimType>gazebo_ros_control/DefaultRobotHWSim</robotSimType>
         </plugin>
-    </gazebo>
+    </gazebo> -->
     <!-- Show the trajectory of trunk center. -->
-    <gazebo>
+    <!-- <gazebo>
         <plugin name="3dplot" filename="libLinkPlot3DPlugin.so">
             <frequency>10</frequency>
@@ -18,5 +18,5 @@
             </plot>
         </plugin>
-    </gazebo>
+    </gazebo> -->
     <!-- Show the trajectory of foot. You can add another trajectory about another foot. -->
     <!-- <gazebo>
@@ -32,6 +32,6 @@
     <gazebo>
         <plugin filename="libgazebo_ros_force.so" name="gazebo_ros_force">
-            <bodyName>trunk</bodyName>
-            <topicName>/apply_force/trunk</topicName>
+            <link_name>base</link_name>
+            <force_frame>world</force_frame>
         </plugin>
     </gazebo>
@@ -44,4 +44,5 @@
             <topic>__default_topic__</topic>
             <plugin filename="libgazebo_ros_imu_sensor.so" name="imu_plugin">
+                <initial_orientation_as_reference>false</initial_orientation_as_reference>
                 <topicName>trunk_imu</topicName>
                 <bodyName>imu_link</bodyName>
@@ -56,5 +57,5 @@
     </gazebo>
     <!-- Foot contacts. -->
-    <gazebo reference="FR_calf">
+    <!-- <gazebo reference="FR_calf">
         <sensor name="FR_foot_contact" type="contact">
         <update_rate>100</update_rate>
@@ -91,7 +92,7 @@
         </contact>
         </sensor>
-    </gazebo>
+    </gazebo> -->
     <!-- Visualization of Foot contacts. -->
-    <gazebo reference="FR_foot">
+    <!-- <gazebo reference="FR_foot">
         <visual>
             <plugin name="drawForcePlugin" filename="libunitreeDrawForcePlugin.so">
@@ -120,5 +121,5 @@
             </plugin>
         </visual>
-    </gazebo>
+    </gazebo> -->
     <gazebo reference="base">
         <material>Gazebo/Green</material>

File: a1_description/xacro/robot.xacro (robot description, xacro)
@@ -5,7 +5,7 @@
     <xacro:include filename="$(find a1_description)/xacro/materials.xacro"/>
     <xacro:include filename="$(find a1_description)/xacro/leg.xacro"/>
-    <!-- <xacro:include filename="$(find a1_description)/xacro/stairs.xacro"/>
+    <!-- <xacro:include filename="$(find a1_description)/xacro/stairs.xacro"/> -->
     <xacro:include filename="$(find a1_description)/xacro/gazebo.xacro"/>
-    <xacro:include filename="$(find a1_gazebo)/launch/stairs.urdf.xacro"/> -->
+    <!-- <xacro:include filename="$(find a1_gazebo)/launch/stairs.urdf.xacro"/> -->
     <!-- <xacro:stairs stairs="15" xpos="0" ypos="0" zpos="0" /> -->
     <!-- Rollover Protection mode will add an additional stick on the top, use "true" or "false" to switch it. -->
@@ -37,5 +37,5 @@
             <origin rpy="0 0 0" xyz="0 0 0"/>
             <geometry>
-                <mesh filename="package://a1_description/meshes/trunk.dae" scale="1 1 1"/>
+                <mesh filename="file://$(find a1_description)/meshes/trunk.dae" scale="1 1 1"/>
             </geometry>
             <material name="orange"/>
